File: shematics_and_layouts/cube/cube.brd (EAGLE design)
At the start: 71 x 69 mm, 13 parts, among them X1 LEDs, X2 BAT

Commit message: TASK: Add switch to cube
Parts:
- added S1: (no value), switch-e-switch:EG1218
- moved X1 17.8 mm to (20.3, 57.1)
- moved B+ 7.62 mm to (62.4, 28.6)
- moved B- 7.62 mm to (54.9, 28.6)
- moved OUT+ 7.62 mm to (65.5, 28.6)
- moved OUT- 7.62 mm to (51.7, 28.6)
- moved + 7.62 mm to (65.5, 51.3)
- moved - 7.62 mm to (51.7, 51.3)
- moved X2 7.62 mm to (58.4, 16.5)
Connections:
- new net N$3: S1.3, VIN+.MP
- net N$1: now also S1.2; no longer VIN+.MP
Routing:
- net N$3: track 0.00 -> 61.7 mm
- net N$1: track 82.0 -> 61.4 mm
- net GND: track 83.2 -> 65.4 mm
- net VCC: track 82.7 -> 64.9 mm
- net N$12: track 54.2 -> 67.9 mm
- net N$2: track 38.5 -> 30.9 mm
