File: shematics_and_layouts/cube/cube.sch (EAGLE design)
At the start: 23 parts, among them K1 LD1117AV33, X1 LEDs

Commit message: TASK: Board outlines for U-Suply components
Parts:
- removed A2: ESP8266, con-lstb:MA04-2
- removed A3: MPU-6050, con-lsta:FE08-1
- removed C1, C2: 100n, rcl:C-EU050-024X044
- removed K1: LD1117AV33, linear:7805T
- removed R1: 10K, rcl:R-EU_0207/10
- removed R2: 1K, rcl:R-EU_0207/10
- removed R3: 2K, rcl:R-EU_0207/10
- removed R4: RGP10M, diode:1N4446
Connections:
- removed net N$10: A1.A4, A3.4
- removed net N$11: A1.A5, A3.3
- removed net N$3: A2.2, C2.1, K1.VO, R1.1, R4.A
- removed net N$4: A2.1, R2.2, R3.1
- removed net N$5: A2.6, R1.2
- removed net N$6: A1.D2, A2.8
- removed net N$8: A1.D3, R2.1
- net GND: no longer A2.7, A3.2, C1.2, C2.2, K1.GND, R3.2
- net VCC: now also A1.RAW; no longer A1.5.5V, A3.1, C1.1, K1.VI, R4.C
Changed lines of the file:
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@@
 <parts>
 <part name="A1" library="Arduino-clone" deviceset="NANO" device=""/>
-<part name="GND1" library="supply1" deviceset="GND" device=""/>
-<part name="A2" library="con-lstb" deviceset="MA04-2" device="" value="ESP8266"/>
-<part name="K1" library="linear" deviceset="78*" device="T" technology="05" value="LD1117AV33"/>
-<part name="R1" library="rcl" deviceset="R-EU_" device="0207/10" value="10K"/>
-<part name="R2" library="rcl" deviceset="R-EU_" device="0207/10" value="1K"/>
-<part name="R3" library="rcl" deviceset="R-EU_" device="0207/10" value="2K"/>
-<part name="R4" library="diode" deviceset="1N4446" device="" value="RGP10M"/>
-<part name="C1" library="rcl" deviceset="C-EU" device="050-024X044" value="100n"/>
-<part name="C2" library="rcl" deviceset="C-EU" device="050-024X044" value="100n"/>
 <part name="VOUT+" library="solpad" deviceset="MCS08" device=""/>
 <part name="VOUT-" library="solpad" deviceset="MCS08" device=""/>
@@
 <part name="BH+" library="solpad" deviceset="MCS08" device=""/>
 <part name="BH-" library="solpad" deviceset="MCS08" device=""/>
-<part name="A3" library="con-lsta" deviceset="FE08-1" device="" value="MPU-6050"/>
-<part name="P+3" library="supply1" deviceset="VCC" device="" value="VCC +5V"/>
-<part name="GND4" library="supply1" deviceset="GND" device=""/>
 <part name="X1" library="con-lstb" deviceset="MA03-1" device="" value="LEDs"/>
 <part name="P+4" library="supply1" deviceset="VCC" device="" value="VCC +5V"/>
@@
 <instances>
 <instance part="A1" gate="G$1" x="-15.24" y="55.88" smashed="yes"/>
-<instance part="GND1" gate="1" x="106.68" y="99.06"/>
-<instance part="A2" gate="G$1" x="71.12" y="124.46"/>
-<instance part="K1" gate="A1" x="25.4" y="119.38"/>
-<instance part="R1" gate="G$1" x="50.8" y="127" rot="R90"/>
-<instance part="R2" gate="G$1" x="71.12" y="106.68"/>
-<instance part="R3" gate="G$1" x="91.44" y="106.68"/>
-<instance part="R4" gate="1" x="25.4" y="132.08" rot="R180"/>
-<instance part="C1" gate="G$1" x="12.7" y="109.22"/>
-<instance part="C2" gate="G$1" x="38.1" y="109.22"/>
 <instance part="VOUT+" gate="G$1" x="-10.16" y="119.38" smashed="yes" rot="R90">
 <attribute name="NAME" x="-13.97" y="121.539" size="1.778" layer="95" rot="R180"/>
@@
 <attribute name="NAME" x="-64.77" y="149.479" size="1.778" layer="95" rot="R180"/>
 </instance>
-<instance part="A3" gate="G$1" x="-93.98" y="63.5"/>
-<instance part="P+3" gate="VCC" x="-83.82" y="81.28"/>
-<instance part="GND4" gate="1" x="-81.28" y="48.26"/>
 <instance part="X1" gate="G$1" x="38.1" y="66.04" rot="R180"/>
 <instance part="P+4" gate="VCC" x="27.94" y="76.2"/>
@@
 <net name="GND" class="0">
 <segment>
-<pinref part="A2" gate="G$1" pin="7"/>
-<wire x1="78.74" y1="127" x2="106.68" y2="127" width="0.1524" layer="91"/>
-<pinref part="GND1" gate="1" pin="GND"/>
-<wire x1="106.68" y1="127" x2="106.68" y2="106.68" width="0.1524" layer="91"/>
-<pinref part="R3" gate="G$1" pin="2"/>
-<wire x1="106.68" y1="106.68" x2="106.68" y2="101.6" width="0.1524" layer="91"/>
-<wire x1="96.52" y1="106.68" x2="106.68" y2="106.68" width="0.1524" layer="91"/>
-<junction x="106.68" y="106.68"/>
-</segment>
-<segment>
-<pinref part="C1" gate="G$1" pin="2"/>
-<wire x1="12.7" y1="104.14" x2="12.7" y2="99.06" width="0.1524" layer="91"/>
-<wire x1="12.7" y1="99.06" x2="25.4" y2="99.06" width="0.1524" layer="91"/>
-<pinref part="C2" gate="G$1" pin="2"/>
-<wire x1="25.4" y1="99.06" x2="38.1" y2="99.06" width="0.1524" layer="91"/>
-<wire x1="38.1" y1="99.06" x2="38.1" y2="104.14" width="0.1524" layer="91"/>
-<pinref part="K1" gate="A1" pin="GND"/>
-<wire x1="25.4" y1="111.76" x2="25.4" y2="99.06" width="0.1524" layer="91"/>
-<junction x="25.4" y="99.06"/>
 <pinref part="VOUT-" gate="G$1" pin="MP"/>
 <wire x1="-7.62" y1="114.3" x2="2.54" y2="114.3" width="0.1524" layer="91"/>
-<wire x1="2.54" y1="114.3" x2="2.54" y2="99.06" width="0.1524" layer="91"/>
-<wire x1="2.54" y1="99.06" x2="12.7" y2="99.06" width="0.1524" layer="91"/>
-<junction x="12.7" y="99.06"/>
+<wire x1="2.54" y1="114.3" x2="2.54" y2="96.52" width="0.1524" layer="91"/>
 <pinref part="GND2" gate="1" pin="GND"/>
-<wire x1="2.54" y1="99.06" x2="2.54" y2="96.52" width="0.1524" layer="91"/>
-<junction x="2.54" y="99.06"/>
 </segment>
 <segment>
@@
 </segment>
 <segment>
-<pinref part="A3" gate="G$1" pin="2"/>
-<wire x1="-86.36" y1="58.42" x2="-81.28" y2="58.42" width="0.1524" layer="91"/>
-<pinref part="GND4" gate="1" pin="GND"/>
-<wire x1="-81.28" y1="58.42" x2="-81.28" y2="50.8" width="0.1524" layer="91"/>
-</segment>
-<segment>
 <pinref part="X1" gate="G$1" pin="3"/>
 <wire x1="30.48" y1="63.5" x2="27.94" y2="63.5" width="0.1524" layer="91"/>
@@
 </segment>
 </net>
-<net name="N$3" class="0">
-<segment>
-<pinref part="R4" gate="1" pin="A"/>
-<wire x1="27.94" y1="132.08" x2="38.1" y2="132.08" width="0.1524" layer="91"/>
-<wire x1="38.1" y1="132.08" x2="38.1" y2="119.38" width="0.1524" layer="91"/>
-<pinref part="K1" gate="A1" pin="VO"/>
-<wire x1="38.1" y1="119.38" x2="35.56" y2="119.38" width="0.1524" layer="91"/>
-<pinref part="C2" gate="G$1" pin="1"/>
-<wire x1="38.1" y1="119.38" x2="38.1" y2="111.76" width="0.1524" layer="91"/>
-<junction x="38.1" y="119.38"/>
-<pinref part="A2" gate="G$1" pin="2"/>
-<wire x1="63.5" y1="119.38" x2="50.8" y2="119.38" width="0.1524" layer="91"/>
-<pinref part="R1" gate="G$1" pin="1"/>
-<wire x1="50.8" y1="119.38" x2="38.1" y2="119.38" width="0.1524" layer="91"/>
-<wire x1="50.8" y1="121.92" x2="50.8" y2="119.38" width="0.1524" layer="91"/>
-<junction x="50.8" y="119.38"/>
-</segment>
-</net>
-<net name="N$4" class="0">
-<segment>
-<pinref part="R2" gate="G$1" pin="2"/>
-<pinref part="R3" gate="G$1" pin="1"/>
-<wire x1="76.2" y1="106.68" x2="81.28" y2="106.68" width="0.1524" layer="91"/>
-<pinref part="A2" gate="G$1" pin="1"/>
-<wire x1="81.28" y1="106.68" x2="86.36" y2="106.68" width="0.1524" layer="91"/>
-<wire x1="78.74" y1="119.38" x2="81.28" y2="119.38" width="0.1524" layer="91"/>
-<wire x1="81.28" y1="119.38" x2="81.28" y2="106.68" width="0.1524" layer="91"/>
-<junction x="81.28" y="106.68"/>
-</segment>
-</net>
-<net name="N$5" class="0">
-<segment>
-<pinref part="R1" gate="G$1" pin="2"/>
-<wire x1="50.8" y1="132.08" x2="60.96" y2="132.08" width="0.1524" layer="91"/>
-<wire x1="60.96" y1="132.08" x2="60.96" y2="124.46" width="0.1524" layer="91"/>
-<pinref part="A2" gate="G$1" pin="6"/>
-<wire x1="60.96" y1="124.46" x2="63.5" y2="124.46" width="0.1524" layer="91"/>
-</segment>
-</net>
-<net name="N$6" class="0">
-<segment>
-<pinref part="A2" gate="G$1" pin="8"/>
-<wire x1="63.5" y1="127" x2="55.88" y2="127" width="0.1524" layer="91"/>
-<wire x1="55.88" y1="127" x2="55.88" y2="45.72" width="0.1524" layer="91"/>
-<pinref part="A1" gate="G$1" pin="D2"/>
-<wire x1="-5.08" y1="45.72" x2="55.88" y2="45.72" width="0.1524" layer="91"/>
-</segment>
-</net>
-<net name="N$8" class="0">
-<segment>
-<pinref part="A1" gate="G$1" pin="D3"/>
-<wire x1="-5.08" y1="48.26" x2="58.42" y2="48.26" width="0.1524" layer="91"/>
-<wire x1="58.42" y1="48.26" x2="58.42" y2="106.68" width="0.1524" layer="91"/>
-<pinref part="R2" gate="G$1" pin="1"/>
-<wire x1="58.42" y1="106.68" x2="66.04" y2="106.68" width="0.1524" layer="91"/>
-</segment>
-</net>
 <net name="VCC" class="0">
 <segment>
-<pinref part="K1" gate="A1" pin="VI"/>
-<wire x1="15.24" y1="119.38" x2="12.7" y2="119.38" width="0.1524" layer="91"/>
-<wire x1="12.7" y1="119.38" x2="12.7" y2="132.08" width="0.1524" layer="91"/>
-<pinref part="R4" gate="1" pin="C"/>
-<wire x1="12.7" y1="132.08" x2="22.86" y2="132.08" width="0.1524" layer="91"/>
-<pinref part="C1" gate="G$1" pin="1"/>
-<wire x1="12.7" y1="119.38" x2="12.7" y2="111.76" width="0.1524" layer="91"/>
-<junction x="12.7" y="119.38"/>
+<pinref part="P+1" gate="VCC" pin="VCC"/>
+<wire x1="2.54" y1="134.62" x2="2.54" y2="119.38" width="0.1524" layer="91"/>
 <pinref part="VOUT+" gate="G$1" pin="MP"/>
 <wire x1="-7.62" y1="119.38" x2="2.54" y2="119.38" width="0.1524" layer="91"/>
-<pinref part="P+1" gate="VCC" pin="VCC"/>
-<wire x1="2.54" y1="119.38" x2="12.7" y2="119.38" width="0.1524" layer="91"/>
-<wire x1="2.54" y1="134.62" x2="2.54" y2="119.38" width="0.1524" layer="91"/>
-<junction x="2.54" y="119.38"/>
 </segment>
 <segment>
 <pinref part="P+2" gate="VCC" pin="VCC"/>
-<wire x1="-60.96" y1="45.72" x2="-60.96" y2="43.18" width="0.1524" layer="91"/>
-<pinref part="A1" gate="G$1" pin="5.5V"/>
-<wire x1="-60.96" y1="43.18" x2="-38.1" y2="43.18" width="0.1524" layer="91"/>
-</segment>
-<segment>
-<pinref part="A3" gate="G$1" pin="1"/>
-<wire x1="-86.36" y1="55.88" x2="-83.82" y2="55.88" width="0.1524" layer="91"/>
-<wire x1="-83.82" y1="55.88" x2="-83.82" y2="78.74" width="0.1524" layer="91"/>
-<pinref part="P+3" gate="VCC" pin="VCC"/>
+<pinref part="A1" gate="G$1" pin="RAW"/>
+<wire x1="-38.1" y1="35.56" x2="-60.96" y2="35.56" width="0.1524" layer="91"/>
+<wire x1="-60.96" y1="35.56" x2="-60.96" y2="45.72" width="0.1524" layer="91"/>
 </segment>
 <segment>
@@
 </segment>
 </net>
-<net name="N$10" class="0">
-<segment>
-<pinref part="A1" gate="G$1" pin="A4"/>
-<wire x1="-38.1" y1="53.34" x2="-43.18" y2="53.34" width="0.1524" layer="91"/>
-<wire x1="-43.18" y1="53.34" x2="-43.18" y2="63.5" width="0.1524" layer="91"/>
-<pinref part="A3" gate="G$1" pin="4"/>
-<wire x1="-43.18" y1="63.5" x2="-86.36" y2="63.5" width="0.1524" layer="91"/>
-</segment>
-</net>
-<net name="N$11" class="0">
-<segment>
-<pinref part="A3" gate="G$1" pin="3"/>
-<wire x1="-86.36" y1="60.96" x2="-45.72" y2="60.96" width="0.1524" layer="91"/>
-<wire x1="-45.72" y1="60.96" x2="-45.72" y2="50.8" width="0.1524" layer="91"/>
-<pinref part="A1" gate="G$1" pin="A5"/>
-<wire x1="-45.72" y1="50.8" x2="-38.1" y2="50.8" width="0.1524" layer="91"/>
-</segment>
-</net>

Commit message: TASK: finished layout Cube
Parts:
- removed BH+, BH-: MCS08, solpad:MCS08
- added X2: BAT, con-lstb:MA03-1
Connections:
- net N$7: now also X2.1; no longer BH-.MP
- net N$9: now also X2.3; no longer BH+.MP
Changed lines of the file:
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@@
 <part name="-" library="solpad" deviceset="MCS08" device=""/>
 <part name="+" library="solpad" deviceset="MCS08" device=""/>
-<part name="BH+" library="solpad" deviceset="MCS08" device=""/>
-<part name="BH-" library="solpad" deviceset="MCS08" device=""/>
 <part name="X1" library="con-lstb" deviceset="MA03-1" device="" value="LEDs"/>
 <part name="P+4" library="supply1" deviceset="VCC" device="" value="VCC +5V"/>
 <part name="GND5" library="supply1" deviceset="GND" device=""/>
+<part name="X2" library="con-lstb" deviceset="MA03-1" device="" value="BAT"/>
 </parts>
 <sheets>
@@
 <wire x1="-73.66" y1="142.24" x2="-73.66" y2="157.48" width="0.1524" layer="94" style="dashdot"/>
 <wire x1="-73.66" y1="157.48" x2="-55.88" y2="157.48" width="0.1524" layer="94" style="dashdot"/>
-<text x="-27.94" y="78.74" size="1.778" layer="95">A1</text>
+<text x="-27.686" y="78.994" size="1.778" layer="95">A1</text>
 </plain>
 <instances>
@@
 <attribute name="NAME" x="-29.21" y="114.681" size="1.778" layer="95"/>
 </instance>
-<instance part="GND2" gate="1" x="2.54" y="93.98"/>
-<instance part="P+1" gate="VCC" x="2.54" y="137.16"/>
-<instance part="P+2" gate="VCC" x="-60.96" y="48.26"/>
-<instance part="GND3" gate="1" x="-55.88" y="10.16"/>
+<instance part="GND2" gate="1" x="2.54" y="93.98" smashed="yes">
+<attribute name="VALUE" x="5.08" y="96.52" size="1.778" layer="96"/>
+</instance>
+<instance part="P+1" gate="VCC" x="2.54" y="137.16" smashed="yes">
+<attribute name="VALUE" x="15.24" y="139.7" size="1.778" layer="96" rot="R180"/>
+</instance>
+<instance part="P+2" gate="VCC" x="-60.96" y="48.26" smashed="yes">
+<attribute name="VALUE" x="-49.276" y="50.8" size="1.778" layer="96" rot="R180"/>
+</instance>
+<instance part="GND3" gate="1" x="-55.88" y="10.16" smashed="yes">
+<attribute name="VALUE" x="-53.34" y="12.7" size="1.778" layer="96"/>
+</instance>
 <instance part="OUT+" gate="G$1" x="-60.96" y="119.38" smashed="yes" rot="R90">
 <attribute name="NAME" x="-64.77" y="121.539" size="1.778" layer="95" rot="R180"/>
@@
 <attribute name="NAME" x="-82.55" y="127.381" size="1.778" layer="95"/>
 </instance>
-<instance part="BH+" gate="G$1" x="-60.96" y="152.4" smashed="yes" rot="R90">
-<attribute name="NAME" x="-64.77" y="154.559" size="1.778" layer="95" rot="R180"/>
+<instance part="X1" gate="G$1" x="38.1" y="66.04" smashed="yes" rot="R180">
+<attribute name="VALUE" x="46.99" y="71.12" size="1.778" layer="96" rot="R180"/>
+<attribute name="NAME" x="44.196" y="73.66" size="1.778" layer="95" rot="R180"/>
 </instance>
-<instance part="BH-" gate="G$1" x="-60.96" y="147.32" smashed="yes" rot="R90">
-<attribute name="NAME" x="-64.77" y="149.479" size="1.778" layer="95" rot="R180"/>
+<instance part="P+4" gate="VCC" x="27.94" y="76.2" smashed="yes">
+<attribute name="VALUE" x="40.132" y="78.74" size="1.778" layer="96" rot="R180"/>
 </instance>
-<instance part="X1" gate="G$1" x="38.1" y="66.04" rot="R180"/>
-<instance part="P+4" gate="VCC" x="27.94" y="76.2"/>
-<instance part="GND5" gate="1" x="27.94" y="55.88"/>
+<instance part="GND5" gate="1" x="27.94" y="55.88" smashed="yes">
+<attribute name="VALUE" x="29.972" y="57.658" size="1.778" layer="96"/>
+</instance>
+<instance part="X2" gate="G$1" x="-66.04" y="149.86" smashed="yes">
+<attribute name="VALUE" x="-72.39" y="149.86" size="1.778" layer="96"/>
+<attribute name="NAME" x="-72.39" y="153.162" size="1.778" layer="95"/>
+</instance>
 </instances>
 <busses>
@@
 <net name="N$7" class="0">
 <segment>
-<pinref part="BH-" gate="G$1" pin="MP"/>
-<wire x1="-58.42" y1="147.32" x2="-50.8" y2="147.32" width="0.1524" layer="91"/>
 <wire x1="-50.8" y1="147.32" x2="-50.8" y2="127" width="0.1524" layer="91"/>
 <pinref part="B-" gate="G$1" pin="MP"/>
 <wire x1="-50.8" y1="127" x2="-58.42" y2="127" width="0.1524" layer="91"/>
+<pinref part="X2" gate="G$1" pin="1"/>
+<wire x1="-50.8" y1="147.32" x2="-58.42" y2="147.32" width="0.1524" layer="91"/>
 </segment>
 </net>
@@
 <wire x1="-58.42" y1="132.08" x2="-45.72" y2="132.08" width="0.1524" layer="91"/>
 <wire x1="-45.72" y1="132.08" x2="-45.72" y2="152.4" width="0.1524" layer="91"/>
-<pinref part="BH+" gate="G$1" pin="MP"/>
-<wire x1="-45.72" y1="152.4" x2="-58.42" y2="152.4" width="0.1524" layer="91"/>
+<pinref part="X2" gate="G$1" pin="3"/>
+<wire x1="-58.42" y1="152.4" x2="-45.72" y2="152.4" width="0.1524" layer="91"/>
 </segment>
 </net>
