File: shematics_and_layouts/column/column.sch (EAGLE design)
At the start: 1 part

Commit message: TASK: col shematic
Parts:
- added X1: (no value), con-conrad:733980-62
- added X2: (no value), con-berg:PN87520
- added X3: (no value), con-lsta:FE05-2
- added X5: LEDs, con-lstb:MA03-1
- renumbered U$1 to A1
Connections:
- new net 3V3@1: A1.3V3@1, X3.5
- new net GND: X1.2, X1.3, X2.4, X5.3
- new net GND@3: A1.GND@1, A1.GND@2, A1.GND@3
- new net GND@7: A1.GND@4, A1.GND@5, A1.GND@6, A1.GND@7, A1.GND@8, X3.6
- new net N$1: A1.GPIO3/SCL1, X3.2
- new net N$2: A1.GPIO2/SDA1, X3.4
- new net N$3: A1.GPIO18, X5.2
- new net VCC: X1.1, X2.1, X5.1
Changed lines of the file:
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@@
 </classes>
 <parts>
-<part name="U$1" library="rpi-zero-without-test-pad" deviceset="RPI-ZERO" device=""/>
+<part name="A1" library="rpi-zero-without-test-pad" deviceset="RPI-ZERO" device=""/>
+<part name="GND1" library="supply1" deviceset="GND" device=""/>
+<part name="P+1" library="supply1" deviceset="VCC" device="" value="VCC +5V"/>
+<part name="X1" library="con-conrad" deviceset="73398?" device="0-62"/>
+<part name="X2" library="con-berg" deviceset="PN87520" device=""/>
+<part name="X3" library="con-lsta" deviceset="FE05-2" device=""/>
+<part name="P+2" library="supply1" deviceset="VCC" device="" value="VCC +5V"/>
+<part name="GND2" library="supply1" deviceset="GND" device=""/>
+<part name="X5" library="con-lstb" deviceset="MA03-1" device="" value="LEDs"/>
+<part name="P+3" library="supply1" deviceset="VCC" device="" value="VCC +5V"/>
+<part name="GND3" library="supply1" deviceset="GND" device=""/>
+<part name="GND5" library="supply1" deviceset="GND" device=""/>
+<part name="GND6" library="supply1" deviceset="GND" device=""/>
 </parts>
 <sheets>
@@
 </plain>
 <instances>
-<instance part="U$1" gate="G$1" x="53.34" y="40.64"/>
+<instance part="A1" gate="G$1" x="53.34" y="40.64"/>
+<instance part="GND1" gate="1" x="27.94" y="104.14" smashed="yes">
+<attribute name="VALUE" x="25.4" y="101.6" size="1.778" layer="96"/>
+</instance>
+<instance part="P+1" gate="VCC" x="27.94" y="121.92" smashed="yes">
+<attribute name="VALUE" x="30.48" y="124.46" size="1.778" layer="96" rot="R180"/>
+</instance>
+<instance part="X1" gate="G$1" x="38.1" y="111.76"/>
+<instance part="X2" gate="G$1" x="114.3" y="96.52"/>
+<instance part="X3" gate="G$1" x="53.34" y="91.44"/>
+<instance part="P+2" gate="VCC" x="109.22" y="106.68" smashed="yes">
+<attribute name="VALUE" x="111.76" y="109.22" size="1.778" layer="96" rot="R180"/>
+</instance>
+<instance part="GND2" gate="1" x="109.22" y="88.9" smashed="yes">
+<attribute name="VALUE" x="106.68" y="86.36" size="1.778" layer="96"/>
+</instance>
+<instance part="X5" gate="G$1" x="114.3" y="58.42" rot="R180"/>
+<instance part="P+3" gate="VCC" x="104.14" y="66.04" smashed="yes">
+<attribute name="VALUE" x="106.68" y="68.58" size="1.778" layer="96" rot="R180"/>
+</instance>
+<instance part="GND3" gate="1" x="104.14" y="50.8" smashed="yes">
+<attribute name="VALUE" x="101.6" y="48.26" size="1.778" layer="96"/>
+</instance>
+<instance part="GND5" gate="1" x="83.82" y="15.24" smashed="yes">
+<attribute name="VALUE" x="81.28" y="12.7" size="1.778" layer="96"/>
+</instance>
+<instance part="GND6" gate="1" x="25.4" y="15.24" smashed="yes">
+<attribute name="VALUE" x="22.86" y="12.7" size="1.778" layer="96"/>
+</instance>
 </instances>
 <busses>
 </busses>
 <nets>
+<net name="VCC" class="0">
+<segment>
+<pinref part="P+1" gate="VCC" pin="VCC"/>
+<wire x1="27.94" y1="114.3" x2="27.94" y2="119.38" width="0.1524" layer="91"/>
+<pinref part="X1" gate="G$1" pin="1"/>
+<wire x1="33.02" y1="114.3" x2="27.94" y2="114.3" width="0.1524" layer="91"/>
+</segment>
+<segment>
+<pinref part="P+2" gate="VCC" pin="VCC"/>
+<wire x1="109.22" y1="104.14" x2="109.22" y2="101.6" width="0.1524" layer="91"/>
+<pinref part="X2" gate="G$1" pin="1"/>
+<wire x1="109.22" y1="101.6" x2="111.76" y2="101.6" width="0.1524" layer="91"/>
+</segment>
+<segment>
+<pinref part="X5" gate="G$1" pin="1"/>
+<pinref part="P+3" gate="VCC" pin="VCC"/>
+<wire x1="106.68" y1="60.96" x2="104.14" y2="60.96" width="0.1524" layer="91"/>
+<wire x1="104.14" y1="60.96" x2="104.14" y2="63.5" width="0.1524" layer="91"/>
+</segment>
+</net>
+<net name="GND" class="0">
+<segment>
+<pinref part="GND1" gate="1" pin="GND"/>
+<wire x1="27.94" y1="109.22" x2="27.94" y2="106.68" width="0.1524" layer="91"/>
+<pinref part="X1" gate="G$1" pin="3"/>
+<pinref part="X1" gate="G$1" pin="2"/>
+<wire x1="33.02" y1="111.76" x2="33.02" y2="109.22" width="0.1524" layer="91"/>
+<wire x1="33.02" y1="109.22" x2="27.94" y2="109.22" width="0.1524" layer="91"/>
+<junction x="33.02" y="109.22"/>
+</segment>
+<segment>
+<pinref part="GND2" gate="1" pin="GND"/>
+<wire x1="109.22" y1="91.44" x2="109.22" y2="93.98" width="0.1524" layer="91"/>
+<pinref part="X2" gate="G$1" pin="4"/>
+<wire x1="109.22" y1="93.98" x2="111.76" y2="93.98" width="0.1524" layer="91"/>
+</segment>
+<segment>
+<pinref part="GND3" gate="1" pin="GND"/>
+<wire x1="104.14" y1="53.34" x2="104.14" y2="55.88" width="0.1524" layer="91"/>
+<pinref part="X5" gate="G$1" pin="3"/>
+<wire x1="104.14" y1="55.88" x2="106.68" y2="55.88" width="0.1524" layer="91"/>
+</segment>
+</net>
+<net name="N$1" class="0">
+<segment>
+<pinref part="X3" gate="G$1" pin="2"/>
+<wire x1="60.96" y1="86.36" x2="66.04" y2="86.36" width="0.1524" layer="91"/>
+<wire x1="66.04" y1="86.36" x2="66.04" y2="81.28" width="0.1524" layer="91"/>
+<wire x1="66.04" y1="81.28" x2="22.86" y2="81.28" width="0.1524" layer="91"/>
+<wire x1="22.86" y1="81.28" x2="22.86" y2="66.04" width="0.1524" layer="91"/>
+<pinref part="A1" gate="G$1" pin="GPIO3/SCL1"/>
+<wire x1="22.86" y1="66.04" x2="30.48" y2="66.04" width="0.1524" layer="91"/>
+</segment>
+</net>
+<net name="N$2" class="0">
+<segment>
+<pinref part="X3" gate="G$1" pin="4"/>
+<wire x1="60.96" y1="88.9" x2="68.58" y2="88.9" width="0.1524" layer="91"/>
+<wire x1="68.58" y1="88.9" x2="68.58" y2="78.74" width="0.1524" layer="91"/>
+<wire x1="68.58" y1="78.74" x2="25.4" y2="78.74" width="0.1524" layer="91"/>
+<wire x1="25.4" y1="78.74" x2="25.4" y2="68.58" width="0.1524" layer="91"/>
+<pinref part="A1" gate="G$1" pin="GPIO2/SDA1"/>
+<wire x1="25.4" y1="68.58" x2="30.48" y2="68.58" width="0.1524" layer="91"/>
+</segment>
+</net>
+<net name="3V3@1" class="0">
+<segment>
+<pinref part="X3" gate="G$1" pin="5"/>
+<wire x1="45.72" y1="91.44" x2="27.94" y2="91.44" width="0.1524" layer="91"/>
+<wire x1="27.94" y1="91.44" x2="27.94" y2="71.12" width="0.1524" layer="91"/>
+<pinref part="A1" gate="G$1" pin="3V3@1"/>
+<wire x1="27.94" y1="71.12" x2="30.48" y2="71.12" width="0.1524" layer="91"/>
+</segment>
+</net>
+<net name="N$3" class="0">
+<segment>
+<pinref part="A1" gate="G$1" pin="GPIO18"/>
+<pinref part="X5" gate="G$1" pin="2"/>
+<wire x1="78.74" y1="58.42" x2="106.68" y2="58.42" width="0.1524" layer="91"/>
+</segment>
+</net>
+<net name="GND@3" class="0">
+<segment>
+<pinref part="A1" gate="G$1" pin="GND@1"/>
+<pinref part="GND6" gate="1" pin="GND"/>
+<wire x1="30.48" y1="60.96" x2="25.4" y2="60.96" width="0.1524" layer="91"/>
+<wire x1="25.4" y1="60.96" x2="25.4" y2="40.64" width="0.1524" layer="91"/>
+<pinref part="A1" gate="G$1" pin="GND@2"/>
+<wire x1="25.4" y1="40.64" x2="25.4" y2="22.86" width="0.1524" layer="91"/>
+<wire x1="25.4" y1="22.86" x2="25.4" y2="17.78" width="0.1524" layer="91"/>
+<wire x1="30.48" y1="40.64" x2="25.4" y2="40.64" width="0.1524" layer="91"/>
+<junction x="25.4" y="40.64"/>
+<pinref part="A1" gate="G$1" pin="GND@3"/>
+<wire x1="30.48" y1="22.86" x2="25.4" y2="22.86" width="0.1524" layer="91"/>
+<junction x="25.4" y="22.86"/>
+</segment>
+</net>
+<net name="GND@7" class="0">
+<segment>
+<pinref part="X3" gate="G$1" pin="6"/>
+<wire x1="60.96" y1="91.44" x2="83.82" y2="91.44" width="0.1524" layer="91"/>
+<wire x1="83.82" y1="91.44" x2="83.82" y2="66.04" width="0.1524" layer="91"/>
+<pinref part="A1" gate="G$1" pin="GND@8"/>
+<wire x1="83.82" y1="66.04" x2="78.74" y2="66.04" width="0.1524" layer="91"/>
+<pinref part="GND5" gate="1" pin="GND"/>
+<wire x1="83.82" y1="66.04" x2="83.82" y2="55.88" width="0.1524" layer="91"/>
+<junction x="83.82" y="66.04"/>
+<pinref part="A1" gate="G$1" pin="GND@4"/>
+<wire x1="83.82" y1="55.88" x2="83.82" y2="48.26" width="0.1524" layer="91"/>
+<wire x1="83.82" y1="48.26" x2="83.82" y2="35.56" width="0.1524" layer="91"/>
+<wire x1="83.82" y1="35.56" x2="83.82" y2="30.48" width="0.1524" layer="91"/>
+<wire x1="83.82" y1="30.48" x2="83.82" y2="17.78" width="0.1524" layer="91"/>
+<wire x1="78.74" y1="55.88" x2="83.82" y2="55.88" width="0.1524" layer="91"/>
+<junction x="83.82" y="55.88"/>
+<pinref part="A1" gate="G$1" pin="GND@5"/>
+<wire x1="78.74" y1="48.26" x2="83.82" y2="48.26" width="0.1524" layer="91"/>
+<junction x="83.82" y="48.26"/>
+<pinref part="A1" gate="G$1" pin="GND@6"/>
+<wire x1="78.74" y1="35.56" x2="83.82" y2="35.56" width="0.1524" layer="91"/>
+<junction x="83.82" y="35.56"/>
+<pinref part="A1" gate="G$1" pin="GND@7"/>
+<wire x1="78.74" y1="30.48" x2="83.82" y2="30.48" width="0.1524" layer="91"/>
+<junction x="83.82" y="30.48"/>
+</segment>
+</net>
 </nets>
 </sheet>

Commit message: TASK: Layout col, remove holes in pi
Connections:
- removed net GND@3: A1.GND@1, A1.GND@2, A1.GND@3
- removed net GND@7: A1.GND@4, A1.GND@5, A1.GND@6, A1.GND@7, A1.GND@8, X3.6
- net GND: now also A1.GND@1, A1.GND@2, A1.GND@3, A1.GND@4, A1.GND@5, A1.GND@6, A1.GND@7, A1.GND@8, X3.6
Changed lines of the file:
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@@
 <part name="GND3" library="supply1" deviceset="GND" device=""/>
 <part name="GND5" library="supply1" deviceset="GND" device=""/>
-<part name="GND6" library="supply1" deviceset="GND" device=""/>
+<part name="GND" library="supply1" deviceset="GND" device=""/>
 </parts>
 <sheets>
@@
 <attribute name="VALUE" x="81.28" y="12.7" size="1.778" layer="96"/>
 </instance>
-<instance part="GND6" gate="1" x="25.4" y="15.24" smashed="yes">
+<instance part="GND" gate="1" x="25.4" y="15.24" smashed="yes">
 <attribute name="VALUE" x="22.86" y="12.7" size="1.778" layer="96"/>
 </instance>
@@
 <wire x1="104.14" y1="55.88" x2="106.68" y2="55.88" width="0.1524" layer="91"/>
 </segment>
+<segment>
+<pinref part="X3" gate="G$1" pin="6"/>
+<wire x1="60.96" y1="91.44" x2="83.82" y2="91.44" width="0.1524" layer="91"/>
+<wire x1="83.82" y1="91.44" x2="83.82" y2="66.04" width="0.1524" layer="91"/>
+<pinref part="A1" gate="G$1" pin="GND@8"/>
+<wire x1="83.82" y1="66.04" x2="78.74" y2="66.04" width="0.1524" layer="91"/>
+<pinref part="GND5" gate="1" pin="GND"/>
+<wire x1="83.82" y1="66.04" x2="83.82" y2="55.88" width="0.1524" layer="91"/>
+<junction x="83.82" y="66.04"/>
+<pinref part="A1" gate="G$1" pin="GND@4"/>
+<wire x1="83.82" y1="55.88" x2="83.82" y2="48.26" width="0.1524" layer="91"/>
+<wire x1="83.82" y1="48.26" x2="83.82" y2="35.56" width="0.1524" layer="91"/>
+<wire x1="83.82" y1="35.56" x2="83.82" y2="30.48" width="0.1524" layer="91"/>
+<wire x1="83.82" y1="30.48" x2="83.82" y2="17.78" width="0.1524" layer="91"/>
+<wire x1="78.74" y1="55.88" x2="83.82" y2="55.88" width="0.1524" layer="91"/>
+<junction x="83.82" y="55.88"/>
+<pinref part="A1" gate="G$1" pin="GND@5"/>
+<wire x1="78.74" y1="48.26" x2="83.82" y2="48.26" width="0.1524" layer="91"/>
+<junction x="83.82" y="48.26"/>
+<pinref part="A1" gate="G$1" pin="GND@6"/>
+<wire x1="78.74" y1="35.56" x2="83.82" y2="35.56" width="0.1524" layer="91"/>
+<junction x="83.82" y="35.56"/>
+<pinref part="A1" gate="G$1" pin="GND@7"/>
+<wire x1="78.74" y1="30.48" x2="83.82" y2="30.48" width="0.1524" layer="91"/>
+<junction x="83.82" y="30.48"/>
+</segment>
+<segment>
+<pinref part="A1" gate="G$1" pin="GND@1"/>
+<pinref part="GND" gate="1" pin="GND"/>
+<wire x1="30.48" y1="60.96" x2="25.4" y2="60.96" width="0.1524" layer="91"/>
+<wire x1="25.4" y1="60.96" x2="25.4" y2="40.64" width="0.1524" layer="91"/>
+<pinref part="A1" gate="G$1" pin="GND@2"/>
+<wire x1="25.4" y1="40.64" x2="25.4" y2="22.86" width="0.1524" layer="91"/>
+<wire x1="25.4" y1="22.86" x2="25.4" y2="17.78" width="0.1524" layer="91"/>
+<wire x1="30.48" y1="40.64" x2="25.4" y2="40.64" width="0.1524" layer="91"/>
+<junction x="25.4" y="40.64"/>
+<pinref part="A1" gate="G$1" pin="GND@3"/>
+<wire x1="30.48" y1="22.86" x2="25.4" y2="22.86" width="0.1524" layer="91"/>
+<junction x="25.4" y="22.86"/>
+</segment>
 </net>
 <net name="N$1" class="0">
@@
 </segment>
 </net>
-<net name="GND@3" class="0">
-<segment>
-<pinref part="A1" gate="G$1" pin="GND@1"/>
-<pinref part="GND6" gate="1" pin="GND"/>
-<wire x1="30.48" y1="60.96" x2="25.4" y2="60.96" width="0.1524" layer="91"/>
-<wire x1="25.4" y1="60.96" x2="25.4" y2="40.64" width="0.1524" layer="91"/>
-<pinref part="A1" gate="G$1" pin="GND@2"/>
-<wire x1="25.4" y1="40.64" x2="25.4" y2="22.86" width="0.1524" layer="91"/>
-<wire x1="25.4" y1="22.86" x2="25.4" y2="17.78" width="0.1524" layer="91"/>
-<wire x1="30.48" y1="40.64" x2="25.4" y2="40.64" width="0.1524" layer="91"/>
-<junction x="25.4" y="40.64"/>
-<pinref part="A1" gate="G$1" pin="GND@3"/>
-<wire x1="30.48" y1="22.86" x2="25.4" y2="22.86" width="0.1524" layer="91"/>
-<junction x="25.4" y="22.86"/>
-</segment>
-</net>
-<net name="GND@7" class="0">
-<segment>
-<pinref part="X3" gate="G$1" pin="6"/>
-<wire x1="60.96" y1="91.44" x2="83.82" y2="91.44" width="0.1524" layer="91"/>
-<wire x1="83.82" y1="91.44" x2="83.82" y2="66.04" width="0.1524" layer="91"/>
-<pinref part="A1" gate="G$1" pin="GND@8"/>
-<wire x1="83.82" y1="66.04" x2="78.74" y2="66.04" width="0.1524" layer="91"/>
-<pinref part="GND5" gate="1" pin="GND"/>
-<wire x1="83.82" y1="66.04" x2="83.82" y2="55.88" width="0.1524" layer="91"/>
-<junction x="83.82" y="66.04"/>
-<pinref part="A1" gate="G$1" pin="GND@4"/>
-<wire x1="83.82" y1="55.88" x2="83.82" y2="48.26" width="0.1524" layer="91"/>
-<wire x1="83.82" y1="48.26" x2="83.82" y2="35.56" width="0.1524" layer="91"/>
-<wire x1="83.82" y1="35.56" x2="83.82" y2="30.48" width="0.1524" layer="91"/>
-<wire x1="83.82" y1="30.48" x2="83.82" y2="17.78" width="0.1524" layer="91"/>
-<wire x1="78.74" y1="55.88" x2="83.82" y2="55.88" width="0.1524" layer="91"/>
-<junction x="83.82" y="55.88"/>
-<pinref part="A1" gate="G$1" pin="GND@5"/>
-<wire x1="78.74" y1="48.26" x2="83.82" y2="48.26" width="0.1524" layer="91"/>
-<junction x="83.82" y="48.26"/>
-<pinref part="A1" gate="G$1" pin="GND@6"/>
-<wire x1="78.74" y1="35.56" x2="83.82" y2="35.56" width="0.1524" layer="91"/>
-<junction x="83.82" y="35.56"/>
-<pinref part="A1" gate="G$1" pin="GND@7"/>
-<wire x1="78.74" y1="30.48" x2="83.82" y2="30.48" width="0.1524" layer="91"/>
-<junction x="83.82" y="30.48"/>
-</segment>
-</net>
